File: Hardware/HeatBed/HeatBed.brd (EAGLE design)
At the start: 257.7 x 252 mm, 4 parts

Commit message: upload gerber
Parts:
- added U$4: (no value), ATEAM:CREATABLE_WORD
Other:
- outline, holes or cut-outs redrawn
- board text added: "3.5ohm"
- board text added: "CREATABLE D3 Heat Bed Ver.2.4"
- board text removed: "3.5ohm exp"
- board text removed: "CREATABLE D2 Heat Bed Ver.2.3"
